Commit message: Changed the diffbot_system.cpp to check for only 1 state interface

File: src/diffdrive_arduino/description/ros2_control/diffbot.ros2_control.xacro (robot description, xacro)
@@ -1,5 +1,5 @@
 <?xml version="1.0"?>
 <robot xmlns:xacro="http://www.ros.org/wiki/xacro">
-  <xacro:macro name="diffbot_ros2_control" params="name prefix">
+  <xacro:macro name="diffbot_ros2_control">
     <ros2_control name="${name}" type="system">
       <hardware>
@@ -11,16 +11,14 @@
         <param name="baud_rate">57600</param>
         <param name="timeout_ms">1000</param>
-        <param name="pid_p">20</param>
-        <param name="pid_d">12</param>
-        <param name="pid_i">0</param>
-        <param name="pid_o">50</param>
       </hardware>
-      <joint name="${prefix}left_wheel_joint">
+      <joint name="left_wheel_joint">
         <command_interface name="velocity"/>
         <state_interface name="velocity"/>
+        <state_interface name="position">
       </joint>
-      <joint name="${prefix}right_wheel_joint">
+      <joint name="right_wheel_joint">
         <command_interface name="velocity"/>
         <state_interface name="velocity"/>
+        <state_interface name="position"/>
       </joint>
     </ros2_control>
