Commit message: changed the robot to reflect camera, with simulation now having camera view

File: src/articubot_one/description/camera.xacro (robot description, xacro)
@@ -1,52 +1,54 @@
 <?xml version="1.0"?>
 <robot xmlns:xacro="http://www.ros.org/wiki/xacro" >
-    <joint name="camera_joint" type="fixed">
-        <parent link="chassis"/>
-        <child link="camera_link"/>
-        <origin xyz="0.276 0 0.181" rpy="0 0.18 0"/>
-    </joint>
-    <link name="camera_link">
-        <visual>
-            <geometry>
-                <box size="0.010 0.03 0.03"/>
-            </geometry>
-            <material name="black"/>
-        </visual>
-        <visual>
-            <origin xyz="0 0 -0.05"/>
-            <geometry>
-                <cylinder radius="0.002" length="0.1"/>
-            </geometry>
-            <material name="black"/>
-        </visual>
-    </link>
-    <joint name="camera_optical_joint" type="fixed">
-        <parent link="camera_link"/>
-        <child link="camera_link_optical"/>
-        <origin xyz="0 0 0" rpy="${-pi/2} 0 ${-pi/2}"/>
-    </joint>
-    <link name="camera_link_optical"></link>
-    <gazebo reference="camera_link">
-        <material>Gazebo/Black</material>
-        <sensor name="camera" type="camera">
-            <pose> 0 0 0 0 0 0 </pose>
-            <visualize>true</visualize>
-            <update_rate>10</update_rate>
-            <camera>
-                <horizontal_fov>1.089</horizontal_fov>
-                <image>
-                    <format>R8G8B8</format>
-                    <width>640</width>
-                    <height>480</height>
-                </image>
-                <clip>
-                    <near>0.05</near>
-                    <far>8.0</far>
-                </clip>
-            </camera>
-            <plugin name="camera_controller" filename="libgazebo_ros_camera.so">
-                <frame_name>camera_link_optical</frame_name>
-            </plugin>
-        </sensor>
-    </gazebo>
+    <xacro:macro name="camera_module" params="parent_link">
+        <joint name="camera_joint" type="fixed">
+            <parent link="${parent_link}"/>
+            <child link="camera_link"/>
+            <origin xyz="0.245 0 0.048" rpy="0 0 0"/>
+        </joint>
+        <link name="camera_link">
+            <visual>
+                <geometry>
+                    <box size="0.001 0.024 0.023"/>
+                </geometry>
+                <material name="my_green"/>
+            </visual>
+            <visual>
+                <origin xyz="0.001 0 0" rpy="0 ${pi/2} 0"/>
+                <geometry>
+                    <cylinder radius="0.002" length="0.002"/>
+                </geometry>
+                <material name="my_black"/>
+            </visual>
+        </link>
+        <joint name="camera_optical_joint" type="fixed">
+            <origin xyz="0 0 0" rpy="${-pi/2} 0 ${-pi/2}" />
+            <parent link="camera_link" />
+            <child link="camera_link_optical" />
+        </joint>
+        <link name="camera_link_optical"></link>
+        <gazebo reference="camera_link">
+            <material>Gazebo/Green</material>
+            <sensor name="camera" type="camera">
+                <pose>0 0 0 0 0 0 </pose>
+                <visualize>true</visualize>
+                <update_rate>10 </update_rate>
+                <camera>
+                    <horizontal_fov>1.089</horizontal_fov>
+                    <image>
+                        <format>R8G8B8</format>    <!--8 bit data for each color channel-->
+                        <width>640</width>
+                        <height>480</height>
+                    </image>
+                    <clip>   <!--How near or far can the camera see-->
+                        <near>0.05</near>
+                        <far>8.0</far>
+                    </clip>
+                </camera>
+                <plugin name="camera_controller" filename="libgazebo_ros_camera.so">
+                    <frame_name>camera_link_optical</frame_name>
+                </plugin>
+            </sensor>
+        </gazebo>
+    </xacro:macro>
 </robot>

File: src/articubot_one/description/robot_core.xacro (robot description, xacro)
@@ -3,19 +3,7 @@
     <xacro:include filename="inertial_macros.xacro"/>
     <xacro:include filename="robot_properties.xacro"/>
-    <material name="white">
-        <color rgba="1 1 1 1" />
-    </material>
-    <material name="orange">
-        <color rgba="1 0.3 0.1 1"/>
-    </material>
-    <material name="blue">
-        <color rgba="0.2 0.2 1 1"/>
-    </material>
-    <material name="black">
-        <color rgba="0 0 0 1"/>
-    </material>
-    <material name="red">
-        <color rgba="1 0 0 1"/>
-    </material>
+    <xacro:property name="materials_included" value="false"/>
+    <xacro:include filename="materials.xacro"/>
+    <xacro:include filename="camera.xacro"/>
     <!-- BASE LINK -->
     <link name="base_link">
@@ -41,5 +29,5 @@
                 <box size="${chassis_length} ${chassis_width} ${chassis_height}"/>
             </geometry>
-            <material name="orange"/>
+            <material name="my_orange"/>
         </visual>
         <collision>
@@ -68,5 +56,5 @@
                 <cylinder radius="${wheel_radius}" length="${wheel_thickness}"/>
             </geometry>
-            <material name="blue"/>
+            <material name="my_blue"/>
         </visual>
         <collision>
@@ -94,5 +82,5 @@
                 <cylinder radius="${wheel_radius}" length="${wheel_thickness}"/>
             </geometry>
-            <material name="blue"/>
+            <material name="my_blue"/>
         </visual>
         <collision>
@@ -119,5 +107,5 @@
                 <sphere radius="${caster_wheel_radius}"/>
             </geometry>
-            <material name="white"/>
+            <material name="my_white"/>
         </visual>
         <collision>
@@ -135,4 +123,6 @@
         <mu2 value="0.001"/>
     </gazebo>
+    <!-- CAMERA MODULE  -->
+    <xacro:camera_module parent_link="chassis"/>
     <gazebo>
         <disable_collisions>
