Commit message: Changed launch_sim to include ros_gz bridge and to use gazebo_control, gazebo_control to have joint_state_publisher

File: src/articubot_one/description/gazebo_control.xacro (robot description, xacro)
@@ -19,4 +19,9 @@
             <publish_wheel_tf>true</publish_wheel_tf>
         </plugin>
+        <plugin name="gz::sim::systems::JointStatePublisher" filename="gz-sim-joint-state-publisher-system">
+            <topic>joint_states</topic>
+            <joint_name>left_wheel_joint</joint_name>
+            <joint_name>right_wheel_joint</joint_name>
+        </plugin>
     </gazebo>
 </robot>

File: src/articubot_one/description/lidar.xacro (robot description, xacro)
@@ -1,20 +1,21 @@
 <?xml version="1.0"?>
 <robot xmlns:xacro="http://www.ros.org/wiki/xacro" >
+    <xacro:include filename="robot_properties.xacro"/>
     <joint name="laser_joint" type="fixed">
         <parent link="chassis"/>
         <child link="laser_frame"/>
-        <origin xyz="0.122 0 0.212" rpy="0 0 0"/>
+        <origin xyz="0.175 0 ${chassis_height+0.03}" rpy="0 0 0"/>
     </joint>
     <link name="laser_frame">
         <visual>
             <geometry>
-                <cylinder radius="0.05" length="0.04"/>
+                <cylinder radius="0.0245" length="0.016"/>
             </geometry>
             <material name="black"/>
         </visual>
         <visual>
-            <origin xyz="0 0 -0.05"/>
+            <origin xyz="0 0 -0.019"/>
             <geometry>
-                <cylinder radius="0.01" length="0.1"/>
+                <box size="0.056 0.056 0.022"/>
             </geometry>
             <material name="black"/>
@@ -30,13 +31,12 @@
     </link>
     <gazebo reference="laser_frame">
-        <material>Gazebo/Black</material>
         <sensor name="laser" type="ray">
             <pose> 0 0 0 0 0 0 </pose>
-            <visualize>false</visualize>
+            <visualize>true</visualize>
             <update_rate>10</update_rate>
             <ray>
                 <scan>
                     <horizontal>
-                        <samples>360</samples>
+                        <samples>500</samples>
                         <min_angle>-3.14</min_angle>
                         <max_angle>3.14</max_angle>
@@ -44,6 +44,6 @@
                 </scan>
                 <range>
-                    <min>0.3</min>
-                    <max>12</max>
+                    <min>0.05</min>
+                    <max>6</max>
                 </range>
             </ray>

File: src/articubot_one/description/robot_core.xacro (robot description, xacro)
@@ -6,4 +6,5 @@
     <xacro:include filename="materials.xacro"/>
     <xacro:include filename="camera.xacro"/>
+    <xacro:include filename="lidar.xacro"/>
     <!-- BASE LINK -->
     <link name="base_link">
