Commit message: fixed change in robot urdf, making sure that all reference are to baselink and that the robot is parallel to ground

File: src/articubot_one/description/robot_core.xacro (robot description, xacro)
@@ -22,5 +22,6 @@
         <parent link="base_link"/>
         <child link="chassis"/>
-        <origin xyz="${-wheel_offset_x_from_chassis_link} 0 ${-wheel_offset_z_from_chassis_link}" rpy="0 0 0"/>
+        <origin xyz="${-wheel_offset_x_from_chassis_link} 0 0" rpy="0 0 0"/>
+        <!-- origin xyz="${-wheel_offset_x_from_chassis_link} 0 ${-wheel_offset_z_from_chassis_link}" rpy="0 0 0"/ -->
     </joint>
     <link name="chassis">
@@ -49,5 +50,6 @@
         <parent link="base_link"/>
         <child link="left_wheel"/>
-        <origin xyz="0 ${wheel_offset_y_from_chassis_link} ${-wheel_offset_z_from_chassis_link}" rpy="-${pi/2} 0 0" />
+        <!-- origin xyz="0 ${wheel_offset_y_from_chassis_link} ${-wheel_offset_z_from_chassis_link}" rpy="-${pi/2} 0 0" / -->
+        <origin xyz="0 ${wheel_offset_y_from_chassis_link} 0" rpy="-${pi/2} 0 0" />
         <axis xyz="0 0 1"/>
     </joint>
@@ -75,5 +77,6 @@
         <parent link="base_link"/>
         <child link="right_wheel"/>
-        <origin xyz="0 ${-wheel_offset_y_from_chassis_link} ${-wheel_offset_z_from_chassis_link}" rpy="${pi/2} 0 0" />
+        <!--origin xyz="0 ${-wheel_offset_y_from_chassis_link} ${-wheel_offset_z_from_chassis_link}" rpy="${pi/2} 0 0" / -->
+        <origin xyz="0 ${-wheel_offset_y_from_chassis_link} 0" rpy="${pi/2} 0 0" />
         <axis xyz="0 0 -1"/>
     </joint>
@@ -99,7 +102,8 @@
     <!-- CASTER WHEEL LINK -->
     <joint name="caster_wheel_joint" type="fixed">
-        <parent link="chassis"/>
+        <parent link="base_link"/>
         <child link="caster_wheel"/>
-        <origin xyz="${caster_wheel_offset_x_from_chassis_link} 0 ${-caster_wheel_offset_z_from_chassis_link}"/>
+        <!-- origin xyz="${caster_wheel_offset_x_from_chassis_link} 0 ${-caster_wheel_offset_z_from_chassis_link}"/ -->
+        <origin xyz="${caster_wheel_offset_x_from_base_link} 0 0"/>
     </joint>
     <link name="caster_wheel">

File: src/articubot_one/description/robot_properties.xacro (robot description, xacro)
@@ -14,7 +14,9 @@
     <xacro:property name="wheel_offset_z_from_chassis_link" value="0.065"/>
 <!-- Castor Wheels-->
-    <xacro:property name="caster_wheel_radius" value="0.03"/>
+    <!-- xacro:property name="caster_wheel_radius" value="0.03"/ -->
+    <xacro:property name="caster_wheel_radius" value="0.0335"/>
     <xacro:property name="caster_wheel_mass" value="0.01"/>
-    <xacro:property name="caster_wheel_offset_x_from_chassis_link" value="0.196"/>
-    <xacro:property name="caster_wheel_offset_z_from_chassis_link" value="0.01"/>
+    <xacro:property name="caster_wheel_offset_x_from_base_link" value="0.128"/>
+    <!-- xacro:property name="caster_wheel_offset_x_from_chassis_link" value="0.196"/ -->
+    <!-- xacro:property name="caster_wheel_offset_z_from_chassis_link" value="0.01"/ -->
 </robot>
