Commit message: modified diffdrive arduino and ros2 control for encoder input

File: src/articubot_one/description/lidar.xacro (robot description, xacro)
@@ -21,9 +21,9 @@
             <material name="black"/>
         </visual>
-        <collision>
+        <!-- <collision>
             <geometry>
                 <cylinder radius="0.05" length="0.04"/>
             </geometry>
-        </collision>
+        </collision> -->
         <xacro:inertial_cylinder mass="0.1" length="0.04" radius="0.05">
             <origin xyz="0 0 0" rpy="0 0 0"/>
@@ -50,5 +50,5 @@
             <plugin name="laser_controller" filename="libgazebo_ros_ray_sensor.so">
                 <ros>
-                    <argument>~/out:=scan</argument>
+                    <argument>~/out:=/scan</argument>
                 </ros>
                 <output_type>sensor_msgs/LaserScan</output_type>

File: src/articubot_one/description/ros2_control.xacro (robot description, xacro)
@@ -13,4 +13,5 @@
                 <param name="baud_rate">57600</param>
                 <param name="timeout_ms">1000</param>
+                <param name="enc_counts_per_rev">20</param>
             </hardware>
             <joint name="left_wheel_joint">
